File: kicad/methane_sensor/ngm2611/ngm2611.kicad_sch (KiCad schematic)
At the start: 1 part

Commit message: Updating schematics as I resolder things to the prototype
Parts:
- added ADC1: ~, new_library:ADC_16-bit_ADS1115_breakout, symbol new_library:16-bit_ADC_Soldered
Changed lines of the file:
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@@
+	)
+	(symbol
+		(lib_id "new_library:16-bit_ADC_Soldered")
+		(at 50.8 78.74 0)
+		(unit 1)
+		(exclude_from_sim no)
+		(in_bom yes)
+		(on_board yes)
+		(dnp no)
+		(fields_autoplaced yes)
+		(property "Reference" "ADC1"
+			(at 53.975 74.93 0)
+			(effects
+				(font
+					(size 1.27 1.27)
+				)
+			)
+		)
+		(property "Value" "~"
+			(at 53.975 77.47 0)
+			(effects
+				(font
+					(size 1.27 1.27)
+				)
+			)
+		)
+		(property "Footprint" "new_library:ADC_16-bit_ADS1115_breakout"
+			(at 50.8 78.74 0)
+			(effects
+				(font
+					(size 1.27 1.27)
+				)
+				(hide yes)
+			)
+		)
+		(property "Datasheet" "http://mm.digikey.com/Volume0/opasdata/d220001/medias/docus/5858/333095%20ADC%2016-bit%20ADS1115%204-channel%20with%20PGA%20breakout%20datasheet.pdf"
+			(at 50.8 78.74 0)
+			(effects
+				(font
+					(size 1.27 1.27)
+				)
+				(hide yes)
+			)
+		)
+		(property "Description" ""
+			(at 50.8 78.74 0)
+			(effects
+				(font
+					(size 1.27 1.27)
+				)
+				(hide yes)
+			)
+		)
+		(pin "3"
+		)
+		(pin "4"
+		)
+		(pin "2"
+		)
+		(pin "4"
+		)
+		(pin "5"
+		)
+		(pin "1"
+		)
+		(pin "5"
+		)
+		(pin "3"
+		)
+		(pin "2"
+		)
+		(pin "1"
+		)
+		(instances
+			(project ""
+				(path "/84797165-2629-4d6e-af73-b85496f7831c"
+					(reference "ADC1")
+					(unit 1)
+				)
+			)
+		)
 	)
 	(symbol
