File: kicad/logger_hat/logger_hat/_autosave-logger_hat.kicad_pcb (KiCad board)
At the start: 2 copper layers, 83.8 x 104.1 mm, 22 parts, among them J1 CO2_sensor_conn, J10 Conn_01x04_Pin, J2 5V_sensor_conn, J3 CH4_Sensor_conn, J4 Reed_switch_conn, J5 PWM_output_1, J6 log_switch_conn, J7 PWM_output_2

Commit message: Read work log
Parts:
- removed BUCK_3V3, BUCK_5V6, BUCK_6to9V1: ~, new_library:LM2596_module_amazon
- added J11: 5V6_IN, Connector_JST:JST_XH_B2B-XH-A_1x02_P2.50mm_Vertical, F.Cu at (102.9, 74.9)
- added J12: 12V_IN, Connector_JST:JST_XH_B2B-XH-A_1x02_P2.50mm_Vertical, F.Cu at (115.6, 86.4)
- added J8: 7V_IN, Connector_JST:JST_XH_B2B-XH-A_1x02_P2.50mm_Vertical, F.Cu at (115.6, 74.9)
- added J9: 3V3_IN, Connector_JST:JST_XH_B2B-XH-A_1x02_P2.50mm_Vertical, F.Cu at (102.9, 86.4)
- added REF**: MountingHole_3.2mm_M3, MountingHole:MountingHole_3.2mm_M3, F.Cu at (123.3, 52.8)
- added REF**: MountingHole_3.2mm_M3, MountingHole:MountingHole_3.2mm_M3, F.Cu at (123.3, 145.4)
- added REF**: MountingHole_3.2mm_M3, MountingHole:MountingHole_3.2mm_M3, F.Cu at (30.6, 145.4)
- added REF**: MountingHole_3.2mm_M3, MountingHole:MountingHole_3.2mm_M3, F.Cu at (30.6, 52.8)
- J2: value 5V_sensor_conn -> 3V3_sensor_conn
- J4: value Reed_switch_conn -> SW_RD
- J6: value log_switch_conn -> SW_LOG
- L4931CZ1, L4931CZ50: footprint Package_TO_SOT_THT:TO-92_Inline -> Package_TO_SOT_THT:TO-92_HandSolder
- moved INA228 150.0 mm to (49.8, 108.8), turned to 90 degrees
- moved J1 123.6 mm to (106.7, 61.5), turned to 180 degrees
- moved J2 75.0 mm to (61.0, 61.0)
- moved J3 75.0 mm to (73.7, 61.0)
- moved ADS1115 74.2 mm to (73.3, 78.3)
- moved L4931CZ50 74.1 mm to (85.1, 56.1)
- moved C1 74.1 mm to (81.3, 53.3)
- moved C2 74.1 mm to (91.4, 58.3)
- moved C3 74.1 mm to (91.4, 68.6)
- moved C4 74.1 mm to (81.3, 68.6)
- moved L4931CZ1 74.0 mm to (85.2, 66.4)
- moved RTC1 29.6 mm to (77.9, 104.8)
- moved J5 3.79 mm to (46.6, 55.9)
- moved J6 2.54 mm to (46.6, 64.8)
- moved J10 1.94 mm to (43.4, 93.1), turned to 180 degrees
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Routing:
- net /SCL: track 32.4 -> 192.6 mm
- net /3V3: track 27.3 -> 145.9 mm
- net /SDA: track 36.0 -> 131.4 mm
- net /D5: track 88.4 -> 174.3 mm
- net /V_bat: track 0.00 -> 78.6 mm, vias 0 -> 4
- net /D3: track 88.1 -> 53.0 mm, vias 6 -> 2
- net /D4: track 183.0 -> 149.0 mm
- net /5V6: track 0.00 -> 33.6 mm, vias 0 -> 3
- net /D7: track 175.5 -> 142.2 mm
- net /PWM: track 157.3 -> 126.3 mm
- net +3V3: track 0.00 -> 29.8 mm, vias 0 -> 2
- net /6to9V: track 0.00 -> 18.1 mm
- net /methane_out: track 0.00 -> 17.3 mm
- net +5V: track 0.00 -> 15.7 mm
- net /sensor_out: track 0.00 -> 15.6 mm
- added copper zone on B.Cu, net GND
Other:
- board size 83.8 x 104.1 mm -> 100 x 100 mm
